Commit message: firefly sdf

File: rotors_description/urdf/firefly.xacro (robot description, xacro)
@@ -185,5 +185,5 @@
   </xacro:vertical_rotor>
   <!-- Mount a VI-sensor in front of the Firefly. -->
-  <xacro:vi_sensor_macro
+  <!-- <xacro:vi_sensor_macro
     namespace="${namespace}/vi_sensor"
     parent_link="${namespace}/base_link"
@@ -192,4 +192,4 @@
     enable_ground_truth="true">
     <origin xyz="0.1 0.0 -0.03" rpy="0.0 0.1 0.0" />
-  </xacro:vi_sensor_macro>
+  </xacro:vi_sensor_macro> -->
 </robot>

File: rotors_gazebo/models/rotors_description/urdf/firefly.xacro (robot description, xacro)
@@ -18,5 +18,5 @@
 <robot name="firefly" xmlns:xacro="http://ros.org/wiki/xacro">
   <!-- Properties -->
-  <xacro:property name="namespace" value="" />
+  <xacro:property name="namespace" value="firefly" />
   <xacro:property name="rotor_velocity_slowdown_sim" value="10" />
   <xacro:property name="use_mesh_file" value="true" />

File: rotors_gazebo/models/rotors_description/urdf/firefly_base.xacro (robot description, xacro)
@@ -17,5 +17,7 @@
 -->
 <robot name="firefly" xmlns:xacro="http://ros.org/wiki/xacro">
-  <!-- macros for gazebo plugins, sensors -->
+  <xacro:arg name='mavlink_addr' default='INADDR_ANY' />
+  <xacro:arg name='mavlink_udp_port' default='14560' />
+  <xacro:arg name='visual_material' default='DarkGrey' />
   <xacro:include filename="$(arg rotors_description_dir)/urdf/component_snippets_1.xacro" />
   <!-- Instantiate iris "mechanics" -->
